Commit message: Setup

File: src/my_robot/urdf/my_robot.xacro (robot description, xacro)
@@ -3,5 +3,5 @@
 <xacro:include filename="$(find my_robot)/urdf/my_robot.gazebo" />
   <link name="robot_footprint"></link>
-  <link name='camera'>
+<link name='camera'>
     <inertial>
       <mass value="0.1"/>
@@ -26,11 +26,18 @@
       </geometry>
     </visual>
-  </link>
- <joint type="fixed" name="camera_joint">
+</link>
+<joint type="fixed" name="camera_joint">
     <origin xyz="0.2 0 0" rpy="0 0 0"/>
     <child link="camera"/>
     <parent link="chassis"/>
     <axis xyz="0 1 0" rpy="0 0 0"/>
-   </joint>
+</joint>
+<joint name="camera_optical_joint" type="fixed">
+    <origin xyz="0 0 0" rpy="-1.5707 0 -1.5707"/>
+    <parent link="camera"/>
+    <child link="camera_link_optical"/>
+</joint>
+  <link name="camera_link_optical">
+  </link>
 <link name='hokuyo'>
     <inertial>

Commit message: Finished implementation

File: src/my_robot/urdf/my_robot.xacro (robot description, xacro)
@@ -3,5 +3,5 @@
 <xacro:include filename="$(find my_robot)/urdf/my_robot.gazebo" />
   <link name="robot_footprint"></link>
-<link name='camera'>
+<link name='camera_link'>
     <inertial>
       <mass value="0.1"/>
@@ -29,5 +29,5 @@
 <joint type="fixed" name="camera_joint">
     <origin xyz="0.2 0 0" rpy="0 0 0"/>
-    <child link="camera"/>
+    <child link="camera_link"/>
     <parent link="chassis"/>
     <axis xyz="0 1 0" rpy="0 0 0"/>
@@ -35,5 +35,5 @@
 <joint name="camera_optical_joint" type="fixed">
     <origin xyz="0 0 0" rpy="-1.5707 0 -1.5707"/>
-    <parent link="camera"/>
+    <parent link="camera_link"/>
     <child link="camera_link_optical"/>
 </joint>
@@ -78,5 +78,5 @@
     <material>Gazebo/Blue</material>
 </gazebo>
-<gazebo reference="camera">
+<gazebo reference="camera_link">
     <material>Gazebo/Red</material>
 </gazebo>

Commit message: Attempt fixing topics

File: src/my_robot/urdf/my_robot.xacro (robot description, xacro)
@@ -3,5 +3,5 @@
 <xacro:include filename="$(find my_robot)/urdf/my_robot.gazebo" />
   <link name="robot_footprint"></link>
-<link name='camera_link'>
+<link name='camera'>
     <inertial>
       <mass value="0.1"/>
@@ -29,5 +29,5 @@
 <joint type="fixed" name="camera_joint">
     <origin xyz="0.2 0 0" rpy="0 0 0"/>
-    <child link="camera_link"/>
+    <child link="camera"/>
     <parent link="chassis"/>
     <axis xyz="0 1 0" rpy="0 0 0"/>
@@ -35,5 +35,5 @@
 <joint name="camera_optical_joint" type="fixed">
     <origin xyz="0 0 0" rpy="-1.5707 0 -1.5707"/>
-    <parent link="camera_link"/>
+    <parent link="camera"/>
     <child link="camera_link_optical"/>
 </joint>
